Commit message: fix(sws_160): correct SWK mesh offset to 0.055 with full geometry explanation

File: robot_end_effectors/schunk_tool_changer/sws_160_description/urdf/sws_160.urdf.xacro (robot description, xacro)
@@ -11,19 +11,38 @@
   ============================================================
   All dimensions from official Schunk datasheet (SWS-160):
-    SWK-160 (robot side / master):  Ø217mm × 55.5mm,  mass=6.44kg
-    SWA-160 (tool side / adapter):  Ø217mm × 37.6mm,  mass=2.86kg
+    SWK-160 (robot side / master):  Ø176mm body, Ø217mm outer, mass=6.44kg
+    SWA-160 (tool side / adapter):  Ø176mm body, Ø217mm outer, mass=2.86kg
     Total coupled height:           55.5 + 37.6 = 93.1mm
-  NOTE: STL meshes do not match datasheet dimensions (SWK STL = 100.6mm).
-        Cylinders are used for both visual and collision to ensure accuracy.
-  Geometry convention:
-    - Link origin is at the MOUNTING face (robot-side face, Z=0)
-    - Geometry extends in +Z direction toward the tool
-    - Cylinder center offset = height/2
-  SWK-160:
-    visual/collision center: xyz="0 0 0.02775"  (55.5/2 = 27.75mm)
-    interface joint offset:  xyz="0 0 0.0555"   (full height = 55.5mm)
-  SWA-160:
-    visual/collision center: xyz="0 0 0.0188"   (37.6/2 = 18.8mm)
-    tool_mount joint offset: xyz="0 0 0.0376"   (full height = 37.6mm)
+  STL coordinate system (verified via bounds measurement):
+    SWK: Y=-30 to +70.6 (axial), X=-88 to +88, Z=-108.5 to +108.5
+    SWA: Y=-37.5 to 0 (axial),   X=-88 to +88, Z=-108.5 to +108.5
+    → STL Y is the cylinder axis in both meshes
+  Rotation rpy="${-pi/2} 0 0" maps STL Y → URDF +Z (away from robot):
+    STL X → URDF X
+    STL Y → URDF +Z  (axial, toward tool)
+    STL Z → URDF -Y
+  SWK-160 STL geometry breakdown (from datasheet drawing + bounds):
+    Y = -55.5 to -30.0 : robot wrist attachment plate (embedded in robot flange CAD)
+    Y = -30.0 to   0.0 : robot-side locating features (spigot, bolt bosses)
+    Y =   0.0 to +55.5 : SWK main visible body (matches datasheet 55.5mm height)
+    Y = +55.5 to +70.6 : interface protrusion that mates INTO the SWA
+    Visual offset xyz="0 0 0.055":
+      With rpy="${-pi/2} 0 0", STL Y maps to URDF +Z.
+      Offset of +0.055m shifts the mesh so that STL Y=-55.5mm aligns with
+      URDF Z=0 (tool0 face). This was determined empirically in RViz —
+      the 0.055 value places the SWK main body flush against tool0
+      with attachment geometry naturally hidden inside the robot flange mesh.
+      NOTE: This offset does NOT equal abs(Y_min)=30mm because the STL
+      includes additional robot-wrist adapter plate geometry (Y=-55.5 to -30)
+      that is not part of the SWK itself.
+    Joint offset: 0.0555m = datasheet SWK height
+      The SWK/SWA mating face is at the end of the main body (55.5mm),
+      NOT at the end of the interface protrusion (70.6mm), because the
+      protrusion goes INTO the SWA — the kinematic interface is at 55.5mm.
+  SWA-160 STL geometry breakdown:
+    Y = -37.5 to 0: full SWA body (matches datasheet 37.6mm height)
+    Y = 0: interface face (mates with SWK) → URDF Z=0 at SWK interface ✅
+    Visual offset xyz="0 0 0.000": no offset needed, Y=0 is already at Z=0
+    Joint offset: 0.0376m = datasheet SWA height
 -->
 <robot xmlns:xacro="http://www.ros.org/wiki/xacro">
@@ -34,17 +53,26 @@
   <!-- ========================================================
        SWK-160  —  robot side (master)
-       Mounts on tool0, interface face at Z=+55.5mm
+       Mounts on tool0, SWK/SWA interface face at Z=+55.5mm
+       Attachment geometry (Y<0 in STL) hidden inside robot flange ✅
        ======================================================== -->
   <xacro:macro name="swk_160_robot_side" params="parent prefix">
     <link name="${prefix}swk_160_link">
-      <!-- Cylinder visual using official datasheet dimensions -->
+      <!-- Mesh visual using official Schunk STL.
+           rpy="${-pi/2} 0 0": maps STL Y → URDF +Z (toward tool).
+           xyz="0 0 0.055": empirically determined offset — places SWK main
+           body (55.5mm) outside robot flange. The STL includes extra robot-
+           wrist adapter plate geometry (beyond the 30mm locating features)
+           which is why offset is 0.055 rather than the expected 0.030.
+           Attachment/locating geometry naturally sits inside robot flange. -->
       <visual>
-        <origin xyz="0 0 0.02775" rpy="0 0 0"/>
+        <origin xyz="0 0 0.055" rpy="${-pi/2} 0 0"/>
         <geometry>
-          <cylinder radius="0.1085" length="0.0555"/>
+          <mesh filename="package://sws_160_description/meshes/swk_160_robot_side_bin.stl"
+                scale="0.001 0.001 0.001"/>
         </geometry>
         <material name="schunk_grey"/>
       </visual>
-      <!-- Collision cylinder — identical to visual -->
+      <!-- Collision cylinder: datasheet dimensions for accurate planning
+           center at half of 55.5mm = 27.75mm, length = 55.5mm -->
       <collision>
         <origin xyz="0 0 0.02775" rpy="0 0 0"/>
@@ -67,5 +95,9 @@
       <origin xyz="0 0 0" rpy="0 0 0"/>
     </joint>
-    <!-- Interface frame at the mating face between SWK and SWA -->
+    <!-- Interface frame at SWK/SWA mating face.
+         Offset = datasheet SWK height = 55.5mm.
+         Note: STL extends to Y=70.6mm but the extra 15.1mm is the
+         interface protrusion that goes INTO the SWA — kinematic
+         interface is at 55.5mm, not 70.6mm. -->
     <link name="${prefix}swk_160_interface"/>
     <joint name="${prefix}swk_160_to_interface" type="fixed">
@@ -81,13 +113,19 @@
   <xacro:macro name="swa_160_tool_side" params="parent prefix">
     <link name="${prefix}swa_160_link">
-      <!-- Cylinder visual using official datasheet dimensions -->
+      <!-- Mesh visual using official Schunk STL.
+           rpy="${-pi/2} 0 0": maps STL Y → URDF +Z (toward tool).
+           xyz="0 0 0.000": STL Y=0 is the interface face → already at
+           URDF Z=0, no offset needed. STL Y=-37.5 (tool mount) maps
+           to URDF Z=-37.5mm (pointing back toward robot, inside SWK). -->
       <visual>
-        <origin xyz="0 0 0.0188" rpy="0 0 0"/>
+        <origin xyz="0 0 0.000" rpy="${-pi/2} 0 0"/>
         <geometry>
-          <cylinder radius="0.1085" length="0.0376"/>
+          <mesh filename="package://sws_160_description/meshes/swa_160_tool_side_bin.stl"
+                scale="0.001 0.001 0.001"/>
         </geometry>
         <material name="schunk_grey"/>
       </visual>
-      <!-- Collision cylinder — identical to visual -->
+      <!-- Collision cylinder: datasheet dimensions
+           center at half of 37.6mm = 18.8mm, length = 37.6mm -->
       <collision>
         <origin xyz="0 0 0.0188" rpy="0 0 0"/>
@@ -110,5 +148,6 @@
       <origin xyz="0 0 0" rpy="0 0 0"/>
     </joint>
-    <!-- Tool mount frame at the gripper mating face -->
+    <!-- Tool mount frame at the gripper mating face
+         Offset = datasheet SWA height = 37.6mm -->
     <link name="${prefix}swa_160_tool_mount"/>
     <joint name="${prefix}swa_160_to_tool_mount" type="fixed">

Commit message: fix(urdf): correct kinect bracket position and orientation on SWK-160 flat face

File: robot_end_effectors/schunk_tool_changer/sws_160_description/urdf/sws_160.urdf.xacro (robot description, xacro)
@@ -42,5 +42,5 @@
   SWA-160 STL geometry breakdown:
     Y = -37.5 to 0: full SWA body (matches datasheet 37.6mm height)
-    Y = 0: interface face (mates with SWK) → URDF Z=0 at SWK interface ✅
+    Y = 0: interface face (mates with SWK) → URDF Z=0 at SWK interface
     Visual offset xyz="0 0 0.000": no offset needed, Y=0 is already at Z=0
     Joint offset: 0.0376m = datasheet SWA height
@@ -54,5 +54,5 @@
        SWK-160  —  robot side (master)
        Mounts on tool0, SWK/SWA interface face at Z=+55.5mm
-       Attachment geometry (Y<0 in STL) hidden inside robot flange ✅
+       Attachment geometry (Y<0 in STL) hidden inside robot flange
        ======================================================== -->
   <xacro:macro name="swk_160_robot_side" params="parent prefix">

File: robot_perception/Azure-Kinect-Sensor-ROS2/abb_kinect_description/urdf/azure_kinect.urdf.xacro (robot description, xacro)
@@ -13,5 +13,5 @@
   ============================================================
   Physical dimensions (Microsoft spec):
-    Body:   126mm x 103mm x 39mm
+    Body:   126mm x 103mm x 39mm  (L x H x D)
     Weight: 440g
   Factory calibration (unit 000720521712):
@@ -19,26 +19,34 @@
     RGB intrinsics:   cx=1021.1, cy=779.0, fx=971.7, fy=971.5
     Depth-to-RGB translation: -32.007mm, -1.871mm, 3.883mm
+  Coordinate convention:
+    camera_base origin = bottom-left-back corner of camera body
+    X = along long axis (126mm direction)
+    Y = up (103mm direction)
+    Z = forward (39mm depth direction, lens faces +Z)
   Frame conventions (ROS standard):
-    camera_base             : origin at bottom-center of camera body
-    depth_camera_frame      : depth sensor center
-    depth_camera_optical_frame : ROS optical frame (Z fwd, X right, Y down)
-    rgb_camera_frame        : RGB sensor center
-    rgb_camera_optical_frame   : ROS optical frame (Z fwd, X right, Y down)
-    imu_frame               : IMU sensor center
+    azure_kinect_link           : origin at bottom-left-back corner
+    depth_camera_frame          : depth sensor center
+    depth_camera_optical_frame  : ROS optical (Z fwd, X right, Y down)
+    rgb_camera_frame            : RGB sensor center
+    rgb_camera_optical_frame    : ROS optical (Z fwd, X right, Y down)
+    imu_frame                   : IMU sensor center
 -->
 <robot xmlns:xacro="http://www.ros.org/wiki/xacro">
-  <xacro:macro name="azure_kinect" params="prefix">
-    <link name="${prefix}camera_base">
+  <xacro:macro name="azure_kinect"
+               params="parent prefix mount_x mount_y mount_z
+                       mount_roll mount_pitch mount_yaw">
+    <link name="${prefix}azure_kinect_link">
+      <!-- Camera body: 126mm x 103mm x 39mm, origin at bottom-left-back corner -->
       <visual>
-        <origin xyz="0.063 0 0.0195" rpy="0 0 0"/>
+        <origin xyz="0.063 0.0515 0.0195" rpy="0 0 0"/>
         <geometry>
           <box size="0.126 0.103 0.039"/>
         </geometry>
         <material name="kinect_dark_gray">
-          <color rgba="0.2 0.2 0.2 1.0"/>
+          <color rgba="0.15 0.15 0.15 1.0"/>
         </material>
       </visual>
       <collision>
-        <origin xyz="0.063 0 0.0195" rpy="0 0 0"/>
+        <origin xyz="0.063 0.0515 0.0195" rpy="0 0 0"/>
         <geometry>
           <box size="0.126 0.103 0.039"/>
@@ -47,17 +55,24 @@
       <inertial>
         <mass value="0.440"/>
-        <origin xyz="0.063 0 0.0195" rpy="0 0 0"/>
-        <inertia
-          ixx="0.000419" ixy="0.0" ixz="0.0"
-          iyy="0.000244" iyz="0.0"
-          izz="0.000577"/>
+        <origin xyz="0.063 0.0515 0.0195" rpy="0 0 0"/>
+        <inertia ixx="0.000419" ixy="0.0" ixz="0.0"
+                 iyy="0.000244" iyz="0.0" izz="0.000577"/>
       </inertial>
     </link>
+    <joint name="${prefix}mount_to_kinect" type="fixed">
+      <parent link="${parent}"/>
+      <child link="${prefix}azure_kinect_link"/>
+      <origin xyz="${mount_x} ${mount_y} ${mount_z}"
+              rpy="${mount_roll} ${mount_pitch} ${mount_yaw}"/>
+    </joint>
+    <!-- Depth camera frame: centered on depth sensor -->
+    <link name="${prefix}depth_camera_frame"/>
     <joint name="${prefix}camera_base_to_depth" type="fixed">
-      <parent link="${prefix}camera_base"/>
+      <parent link="${prefix}azure_kinect_link"/>
       <child link="${prefix}depth_camera_frame"/>
       <origin xyz="0.063 0.011 0.020" rpy="0 0 0"/>
     </joint>
-    <link name="${prefix}depth_camera_frame"/>
+    <!-- Depth optical frame: ROS convention (Z fwd, X right, Y down) -->
+    <link name="${prefix}depth_camera_optical_frame"/>
     <joint name="${prefix}depth_camera_frame_to_optical" type="fixed">
       <parent link="${prefix}depth_camera_frame"/>
@@ -65,5 +80,6 @@
       <origin xyz="0 0 0" rpy="${-pi/2} 0 ${-pi/2}"/>
     </joint>
-    <link name="${prefix}depth_camera_optical_frame"/>
+    <!-- RGB camera frame: offset from depth by factory calibration -->
+    <link name="${prefix}rgb_camera_frame"/>
     <joint name="${prefix}depth_to_rgb" type="fixed">
       <parent link="${prefix}depth_camera_frame"/>
@@ -71,5 +87,6 @@
       <origin xyz="-0.032007 -0.001871 0.003883" rpy="0 0 0"/>
     </joint>
-    <link name="${prefix}rgb_camera_frame"/>
+    <!-- RGB optical frame: ROS convention (Z fwd, X right, Y down) -->
+    <link name="${prefix}rgb_camera_optical_frame"/>
     <joint name="${prefix}rgb_camera_frame_to_optical" type="fixed">
       <parent link="${prefix}rgb_camera_frame"/>
@@ -77,5 +94,6 @@
       <origin xyz="0 0 0" rpy="${-pi/2} 0 ${-pi/2}"/>
     </joint>
-    <link name="${prefix}rgb_camera_optical_frame"/>
+    <!-- IMU frame: offset from depth by factory calibration -->
+    <link name="${prefix}imu_frame"/>
     <joint name="${prefix}depth_to_imu" type="fixed">
       <parent link="${prefix}depth_camera_frame"/>
@@ -83,5 +101,4 @@
       <origin xyz="-0.050680 0.004068 0.001674" rpy="0 0 0"/>
     </joint>
-    <link name="${prefix}imu_frame"/>
   </xacro:macro>
 </robot>

File: robot_perception/Azure-Kinect-Sensor-ROS2/abb_kinect_description/urdf/eye_in_hand_mount.urdf.xacro (robot description, xacro)
@@ -5,64 +5,97 @@
   File:        eye_in_hand_mount.urdf.xacro
   Description: Eye-in-hand mount macro for Azure Kinect DK
-               on ABB IRB6700. Attaches camera to any parent
-               frame (typically tool0 or gripper body).
+               on ABB IRB6700. Mounts Kinect on aluminum
+               extrusion bracket on flat chamfer face of SWK-160.
   Author:      Farzaneh Eskandari
   Email:       farzane.eskandarii@gmail.com
   Date:        2026-06-05
   ============================================================
-  USAGE in MoveIt config robot.urdf.xacro:
+  Physical setup (from photos 2026-06-17):
+    - Bracket: aluminum T-slot extrusion, L-shaped
+    - Mounted on: flat chamfer face of SWK-160
+    - Bracket extends ~50mm away from SWK flat face
+    - Kinect long axis (126mm) parallel to tool Z axis
+    - Kinect lens faces along tool Z (+Z, toward TCP)
+  Verified SWK local axes (from TF matrix, all joints=0):
+    +X (red)  = pointing DOWN in world (-Z world)
+    +Y (green) = pointing SIDEWAYS
+    +Z (blue) = pointing along TOOL AXIS toward TCP
+    → "away from SWK flat face" = -X direction in SWK local frame
+  Mount parameters (approximate — superseded by hand-eye calibration):
+    mount_x = -0.1085m : SWK outer radius to flat face (108.5mm) in -X
+    mount_z = 0.025m   : mid-SWK body along tool Z axis
+    bracket extends further 50mm in -X from bracket origin
+  NOTE: All values approximate for collision avoidance visualization.
+        Hand-eye calibration provides the accurate camera→robot transform.
+  USAGE in main robot URDF:
     <xacro:include filename="$(find abb_kinect_description)/urdf/eye_in_hand_mount.urdf.xacro"/>
-    <xacro:kinect_eye_in_hand parent="rob1_tool0" prefix="rob1_"/>
-  TO REMOVE CAMERA: comment out those two lines. Nothing else changes.
-  TO MOVE TO GRIPPER: change parent to "rob1_gripper_base_link"
-  Parameters:
-    parent   : parent frame to attach camera to
-    prefix   : TF prefix (e.g. "rob1_")
-    mount_x  : X offset from parent (default 0.0m)
-    mount_y  : Y offset from parent (default 0.0m)
-    mount_z  : Z standoff distance  (default 0.050m = 50mm)
-  NOTE: mount_z is a placeholder — update after physical
-        bracket measurement. After hand-eye calibration
-        (Step 5) this is superseded by calibrated transform.
+    <xacro:kinect_eye_in_hand parent="rob1_swk_160_link" prefix="rob1_"
+        mount_x="-0.1085" mount_y="0.0" mount_z="0.025"
+        mount_roll="0" mount_pitch="0" mount_yaw="0"/>
+  TO REMOVE CAMERA: comment out those two lines.
 -->
 <robot xmlns:xacro="http://www.ros.org/wiki/xacro">
   <xacro:include filename="$(find abb_kinect_description)/urdf/azure_kinect.urdf.xacro"/>
-  <xacro:macro name="kinect_eye_in_hand" params="parent prefix mount_x:=0.0 mount_y:=0.0 mount_z:=0.050">
-    <link name="${prefix}kinect_mount_link">
+  <xacro:macro name="kinect_eye_in_hand"
+               params="parent prefix mount_x mount_y mount_z
+                       mount_roll mount_pitch mount_yaw">
+    <!-- =====================================================
+         Bracket: aluminum T-slot extrusion, L-shaped
+         Sits on flat chamfer face of SWK-160
+         Extends in -X direction (away from SWK flat face)
+         Approximate size: 50mm deep x 60mm wide x 40mm tall
+         ===================================================== -->
+    <link name="${prefix}kinect_bracket">
       <visual>
-        <origin xyz="0 0 ${mount_z/2}" rpy="0 0 0"/>
+        <origin xyz="-0.025 0 0" rpy="0 0 0"/>
         <geometry>
-          <cylinder radius="0.060" length="${mount_z}"/>
+          <box size="0.050 0.060 0.040"/>
         </geometry>
-        <material name="kinect_bracket_grey">
-          <color rgba="0.5 0.5 0.5 0.8"/>
+        <material name="bracket_silver">
+          <color rgba="0.75 0.75 0.75 1.0"/>
         </material>
       </visual>
       <collision>
-        <origin xyz="0 0 ${mount_z/2}" rpy="0 0 0"/>
+        <origin xyz="-0.025 0 0" rpy="0 0 0"/>
         <geometry>
-          <cylinder radius="0.060" length="${mount_z}"/>
+          <box size="0.050 0.060 0.040"/>
         </geometry>
       </collision>
       <inertial>
         <mass value="0.200"/>
-        <origin xyz="0 0 ${mount_z/2}" rpy="0 0 0"/>
-        <inertia
-          ixx="0.000017" ixy="0.0" ixz="0.0"
-          iyy="0.000017" iyz="0.0"
-          izz="0.000036"/>
+        <origin xyz="-0.025 0 0" rpy="0 0 0"/>
+        <inertia ixx="0.0003" iyy="0.0003" izz="0.0003"
+                 ixy="0" ixz="0" iyz="0"/>
       </inertial>
     </link>
-    <joint name="${prefix}tool0_to_kinect_mount" type="fixed">
+    <!-- Attach bracket to SWK flat chamfer face
+         mount_x=-0.1085: SWK outer radius, bracket on flat face
+         mount_z=0.025: mid-SWK body along tool axis -->
+    <joint name="${prefix}swk_to_bracket" type="fixed">
       <parent link="${parent}"/>
-      <child link="${prefix}kinect_mount_link"/>
-      <origin xyz="${mount_x} ${mount_y} ${mount_z}" rpy="0 0 0"/>
+      <child link="${prefix}kinect_bracket"/>
+      <origin xyz="${mount_x} ${mount_y} ${mount_z}"
+              rpy="${mount_roll} ${mount_pitch} ${mount_yaw}"/>
     </joint>
-    <xacro:azure_kinect prefix="${prefix}"/>
-    <joint name="${prefix}kinect_mount_to_camera_base" type="fixed">
-      <parent link="${prefix}kinect_mount_link"/>
-      <child link="${prefix}camera_base"/>
-      <origin xyz="0 0 0" rpy="0 0 0"/>
-    </joint>
+    <!-- =====================================================
+         Kinect: mounted on top of bracket
+         Extends further 50mm in -X from bracket origin
+         Long axis (126mm) along Z (tool axis direction)
+         Lens faces +Z (toward TCP)
+         azure_kinect_link origin = bottom-left-back corner:
+           X = long axis (126mm) → along tool Z → use mount_z
+           Y = height (103mm)    → along world up → use mount_x (negative)
+           Z = depth (39mm)      → lens direction → already +Z
+         ===================================================== -->
+    <xacro:azure_kinect
+      parent="${prefix}kinect_bracket"
+      prefix="${prefix}"
+      mount_x="-0.050"
+      mount_y="-0.0515"
+      mount_z="-0.063"
+      mount_roll="0"
+      mount_pitch="0"
+      mount_yaw="0"
+    />
   </xacro:macro>
 </robot>

Commit message: fix(tool-chain): model full flange-to-tool stack, clocking, and calibrated camera frame
Corrected the kinematic chain between the robot flange and the tool
changer to match the real hardware, and baked the hand-eye calibration
into the URDF as the authoritative camera frame.

Chain (flange outward), now fully modeled:
  tool0
   -> flange adapter plate A (20mm)   [added]
   -> flange adapter plate B (15mm)   [added]
   -> ABB force sensor (62mm)
   -> tool-side adapter plate (4mm)
   -> SWK-160 tool changer (clocked 15 deg about Z)  [clocking modeled]
   -> SWA-160

Changes:
- abb_force_sensor_description: add two missing flange-side adapter
  plates (20mm + 15mm), measured with calipers. Sensor and everything
  above now correctly +35mm from flange. tool0->swk now 0.101m.
- sws_160: add generic straight TCP frame (tcp_straight) that cancels
  the 15 deg changer clocking, giving an un-clocked frame aligned with
  tool0 nominal axes for all tools.
- Bake 20-sample hand-eye calibration into rob1_rgb_camera_optical_frame,
  attached directly to tool0 (translation [-0.148,-0.075,0.162], rot
  ~-74.5 deg about Z). Single authoritative camera frame.
- azure_kinect.urdf.xacro: rename chain optical frame to
  *_optical_frame_visual so the calibrated frame is the sole definition.
- kinect_with_urdf.launch: add static bridge connecting the driver's
  camera tree (camera_base) into the robot tree at the calibrated frame,
  so /points2 renders correctly in world coordinates.
- Add calibration result file (.calib).

File: robot_end_effectors/schunk_tool_changer/sws_160_description/urdf/sws_160.urdf.xacro (robot description, xacro)
@@ -156,4 +156,16 @@
       <origin xyz="0 0 0.0376" rpy="0 0 0"/>
     </joint>
+    <!-- =====================================================
+         Generic STRAIGHT TCP frame at the tool mounting face.
+         Cancels the tool-changer clocking (-15 deg about Z) so
+         the frame axes align with tool0's nominal orientation.
+         Tools add their own length below this frame.
+         ===================================================== -->
+    <link name="${prefix}tcp_straight"/>
+    <joint name="${prefix}tool_mount_to_tcp_straight" type="fixed">
+      <parent link="${prefix}swa_160_tool_mount"/>
+      <child link="${prefix}tcp_straight"/>
+      <origin xyz="0 0 0" rpy="0 0 ${-15*pi/180}"/>
+    </joint>
   </xacro:macro>
 </robot>

File: robot_perception/Azure-Kinect-Sensor-ROS2/abb_kinect_description/urdf/azure_kinect.urdf.xacro (robot description, xacro)
@@ -88,8 +88,8 @@
     </joint>
     <!-- RGB optical frame: ROS convention (Z fwd, X right, Y down) -->
-    <link name="${prefix}rgb_camera_optical_frame"/>
+    <link name="${prefix}rgb_camera_optical_frame_visual"/>
     <joint name="${prefix}rgb_camera_frame_to_optical" type="fixed">
       <parent link="${prefix}rgb_camera_frame"/>
-      <child link="${prefix}rgb_camera_optical_frame"/>
+      <child link="${prefix}rgb_camera_optical_frame_visual"/>
       <origin xyz="0 0 0" rpy="${-pi/2} 0 ${-pi/2}"/>
     </joint>
